File: PCB/Pico2ROMEmuCB1.kicad_sch (KiCad schematic)
At the start: 7 parts, among them CN1 Conn_02x15, CN2 Conn_02x14_Counter_Clockwise, J1 Conn_01x02

Commit message: 修正
Parts:
- removed MOD1: RP2350BCoreBoard, Connector_PinHeader_2.54mm:PinHeader_1x01_P2.54mm_Vertical, symbol Connector_Generic:Conn_01x01
Connections:
- net CE#: now also R2.2; no longer R2.1
- net GPIO23: now also R2.1; no longer R2.2
- no-connect marks 2 -> 1
Other:
- moved on the sheet: R2
Changed lines of the file:
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@@
 		(at 38.1 106.68)
-	)
-	(no_connect
-		(at 191.77 87.63)
 	)
 	(wire
@@
 	)
 	(symbol
-		(lib_id "Connector_Generic:Conn_01x01")
-		(at 196.85 87.63 0)
-		(unit 1)
-		(exclude_from_sim yes)
-		(in_bom no)
-		(on_board yes)
-		(dnp no)
-		(fields_autoplaced yes)
-		(property "Reference" "MOD1"
-			(at 199.39 86.3599 0)
-			(effects
-				(font
-					(size 1.27 1.27)
-				)
-				(justify left)
-			)
-		)
-		(property "Value" "RP2350BCoreBoard"
-			(at 199.39 88.8999 0)
-			(effects
-				(font
-					(size 1.27 1.27)
-				)
-				(justify left)
-			)
-		)
-		(property "Footprint" "Connector_PinHeader_2.54mm:PinHeader_1x01_P2.54mm_Vertical"
-			(at 196.85 87.63 0)
-			(effects
-				(font
-					(size 1.27 1.27)
-				)
-				(hide yes)
-			)
-		)
-		(property "Datasheet" "~"
-			(at 196.85 87.63 0)
-			(effects
-				(font
-					(size 1.27 1.27)
-				)
-				(hide yes)
-			)
-		)
-		(property "Description" "Generic connector, single row, 01x01, script generated (kicad-library-utils/schlib/autogen/connector/)"
-			(at 196.85 87.63 0)
-			(effects
-				(font
-					(size 1.27 1.27)
-				)
-				(hide yes)
-			)
-		)
-		(pin "1"
-		)
-		(instances
-			(project ""
-				(path "/b6e14dc5-2bad-4306-bb64-c2b07cf42bf7"
-					(reference "MOD1")
-					(unit 1)
-				)
-			)
-		)
-	)
-	(symbol
 		(lib_id "power:+5V")
 		(at 68.58 40.64 270)
@@
 	(symbol
 		(lib_id "Device:R_Small_US")
-		(at 76.2 127 90)
+		(at 76.2 127 270)
 		(unit 1)
 		(exclude_from_sim no)
@@
 		(dnp no)
 		(property "Reference" "R2"
-			(at 77.216 124.968 90)
+			(at 75.184 129.032 90)
 			(effects
 				(font
@@
 		)
 		(property "Value" "1k"
-			(at 76.708 129.032 90)
-			(effects
-				(font
+			(at 75.692 124.968 90)
+			(effects
+				(font
